File: SBR_PCB/L298N_Remake.kicad_sch (KiCad schematic)
At the start: 24 parts, among them J1 Conn_01x02, J2 Conn_01x02, U1 L298N, U2 MPU-6050, U3 AMS1117-3.3, U4 LM7812_TO220

Commit message: images are added
Other:
- note added: "DRIVER CONFIGURATION"
- note added: "L98N and MPU6050 Power Regulators"
- moved on the sheet: BT1, C2, C3, C4, D10-MPU6050, D9-L298N1, R1, R2, U3, U4
